File: HARDWARE/Prototipo_1/QR/_autosave-QR.kicad_pcb (KiCad board)
At the start: 2 copper layers, 46.2 x 31.8 mm, 15 parts, among them J1 SEL_POWER, J2 Pulsador, J4 RJ45, J6 TTL, J7 CAM, Q1 MMBT2222L, U1 Max232

Commit message: version_4
Parts:
- moved J2 15.5 mm to (61.7, 60.2), turned to 180 degrees
Routing:
- net (no net): track 0.00 -> 15.2 mm, vias 0 -> 6
- net GND: track 29.4 -> 37.7 mm, vias 6 -> 7
- net /TRIG: track 51.6 -> 58.9 mm
- net /POWER: track 91.7 -> 90.9 mm
Other:
- board size 46.2 x 31.8 mm -> 46.2 x 40 mm
- net class Default: trace_width 0.254 -> 0.5
- board text added: "1"
- board text added: "G"
- board text added: "P"
- board text added: "R"
- board text added: "T"
