File: HARDWARE/Prototipo_1/QR/_saved_QR.sch (KiCad schematic (older format))
At the start: 15 parts, among them J1 SEL_POWER, J2 Pulsador, J4 RJ45, J6 TTL, J7 CAM, Q1 MMBT2222L, U1 Max232

Commit message: version_4
Parts:
- D1: footprint LEDs:LED_0603 -> LEDs:LED_0805_HandSoldering
- J6: footprint (none) -> Socket_Strips:Socket_Strip_Straight_1x04_Pitch2.54mm
Connections:
- net +5V: no longer R3.1
- net POWER: now also R3.1
Changed lines of the file:
@@
 F 0 "D1" H 2050 3850 50  0000 C CNN
 F 1 "LED" H 2050 3650 50  0000 C CNN
-F 2 "LEDs:LED_0603" H 2050 3750 50  0001 C CNN
+F 2 "LEDs:LED_0805_HandSoldering" H 2050 3750 50  0001 C CNN
 F 3 "" H 2050 3750 50  0001 C CNN
 	1    2050 3750
@@
 Wire Wire Line
 	2050 3200 2050 3050
-$Comp
-L +5V #PWR05
-U 1 1 595DFAA7
-P 2400 2900
-F 0 "#PWR05" H 2400 2750 50  0001 C CNN
-F 1 "+5V" H 2400 3040 50  0000 C CNN
-F 2 "" H 2400 2900 50  0001 C CNN
-F 3 "" H 2400 2900 50  0001 C CNN
-	1    2400 2900
-	1    0    0    -1
-$EndComp
 Wire Wire Line
 	1300 4250 1100 4250
@@
 $EndComp
 $Comp
-L +3.3V #PWR06
+L +3.3V #PWR05
 U 1 1 595E0426
 P 5800 1750
-F 0 "#PWR06" H 5800 1600 50  0001 C CNN
+F 0 "#PWR05" H 5800 1600 50  0001 C CNN
 F 1 "+3.3V" H 5800 1890 50  0000 C CNN
 F 2 "" H 5800 1750 50  0001 C CNN
@@
 NoConn ~ 4650 1750
 $Comp
-L GND #PWR07
+L GND #PWR06
 U 1 1 595E04F7
 P 4750 1950
-F 0 "#PWR07" H 4750 1700 50  0001 C CNN
+F 0 "#PWR06" H 4750 1700 50  0001 C CNN
 F 1 "GND" H 4750 1800 50  0000 C CNN
 F 2 "" H 4750 1950 50  0001 C CNN
@@
 	6150 2050 6150 1750
 $Comp
-L +5V #PWR08
+L +5V #PWR07
 U 1 1 595E0702
 P 6150 1750
-F 0 "#PWR08" H 6150 1600 50  0001 C CNN
+F 0 "#PWR07" H 6150 1600 50  0001 C CNN
 F 1 "+5V" H 6150 1890 50  0000 C CNN
 F 2 "" H 6150 1750 50  0001 C CNN
@@
 POWER
 $Comp
-L GND #PWR09
+L GND #PWR08
 U 1 1 595E4BA1
 P 10300 1500
-F 0 "#PWR09" H 10300 1250 50  0001 C CNN
+F 0 "#PWR08" H 10300 1250 50  0001 C CNN
 F 1 "GND" H 10300 1350 50  0000 C CNN
 F 2 "" H 10300 1500 50  0001 C CNN
@@
 $EndComp
 $Comp
-L GND #PWR010
+L GND #PWR09
 U 1 1 595E561A
 P 7400 2600
-F 0 "#PWR010" H 7400 2350 50  0001 C CNN
+F 0 "#PWR09" H 7400 2350 50  0001 C CNN
 F 1 "GND" H 7400 2450 50  0000 C CNN
 F 2 "" H 7400 2600 50  0001 C CNN
@@
 	7400 2550 7400 2600
 $Comp
-L GND #PWR011
+L GND #PWR010
 U 1 1 595E6D0B
 P 2050 4750
-F 0 "#PWR011" H 2050 4500 50  0001 C CNN
+F 0 "#PWR010" H 2050 4500 50  0001 C CNN
 F 1 "GND" H 2050 4600 50  0000 C CNN
 F 2 "" H 2050 4750 50  0001 C CNN
@@
 F 0 "J6" H 4150 3400 50  0000 C CNN
 F 1 "TTL" V 4250 3150 50  0000 C CNN
-F 2 "" H 4150 3150 50  0001 C CNN
+F 2 "Socket_Strips:Socket_Strip_Straight_1x04_Pitch2.54mm" H 4150 3150 50  0001 C CNN
 F 3 "" H 4150 3150 50  0001 C CNN
 	1    4150 3150
@@
 Wire Wire Line
 	2400 3050 2050 3050
+Text Label 2400 2900 0    60   ~ 0
+POWER
 $EndSCHEMATC
